Commit message: Update src folder with latest

File: src/ur5_description/urdf/ur5.urdf.xacro (robot description, xacro)
@@ -4,269 +4,4 @@
     <xacro:include filename="ur5_gazebo.xacro" />
     <xacro:include filename="ur5_ros2_control.xacro" />
-    <link name="base_link" />
-    <link name="base_link_inertia">
-        <visual>
-            <origin rpy="0 0 3.141592653589793" xyz="0 0 0" />
-            <geometry>
-                <mesh filename="package://ur5_description/visual/base.dae" />
-            </geometry>
-            <material name="LightGrey">
-                <color rgba="0.7 0.7 0.7 1.0" />
-            </material>
-        </visual>
-        <collision>
-            <origin rpy="0 0 3.141592653589793" xyz="0 0 0" />
-            <geometry>
-                <mesh filename="package://ur5_description/collision/base.stl" />
-            </geometry>
-        </collision>
-        <inertial>
-            <mass value="4.0" />
-            <origin rpy="0 0 0" xyz="0 0 0" />
-            <inertia ixx="0.00443333156" ixy="0.0" ixz="0.0" iyy="0.00443333156" iyz="0.0" izz="0.0072" />
-        </inertial>
-    </link>
-    <link name="shoulder_link">
-        <visual>
-            <origin rpy="0 0 3.141592653589793" xyz="0 0 0" />
-            <geometry>
-                <mesh filename="package://ur5_description/visual/shoulder.dae" />
-            </geometry>
-            <material name="LightGrey">
-                <color rgba="0.7 0.7 0.7 1.0" />
-            </material>
-        </visual>
-        <collision>
-            <origin rpy="0 0 3.141592653589793" xyz="0 0 0" />
-            <geometry>
-                <mesh filename="package://ur5_description/collision/shoulder.stl" />
-            </geometry>
-        </collision>
-        <inertial>
-            <mass value="3.7" />
-            <origin rpy="0 0 0" xyz="0 0 0" />
-            <inertia ixx="0.014972352344389999" ixy="0.0" ixz="0.0" iyy="0.014972352344389999" iyz="0.0" izz="0.01040625" />
-        </inertial>
-    </link>
-    <link name="upper_arm_link">
-        <visual>
-            <origin rpy="1.5707963267948966 0 -1.5707963267948966" xyz="0 0 0.13585" />
-            <geometry>
-                <mesh filename="package://ur5_description/visual/upperarm.dae" />
-            </geometry>
-            <material name="LightGrey">
-                <color rgba="0.7 0.7 0.7 1.0" />
-            </material>
-        </visual>
-        <collision>
-            <origin rpy="1.5707963267948966 0 -1.5707963267948966" xyz="0 0 0.13585" />
-            <geometry>
-                <mesh filename="package://ur5_description/collision/upperarm.stl" />
-            </geometry>
-        </collision>
-        <inertial>
-            <mass value="8.393" />
-            <origin rpy="0 1.5707963267948966 0" xyz="-0.2125 0.0 0.136" />
-            <inertia ixx="0.1338857818623325" ixy="0.0" ixz="0.0" iyy="0.1338857818623325" iyz="0.0" izz="0.0151074" />
-        </inertial>
-    </link>
-    <link name="forearm_link">
-        <visual>
-            <origin rpy="1.5707963267948966 0 -1.5707963267948966" xyz="0 0 0.0165" />
-            <geometry>
-                <mesh filename="package://ur5_description/visual/forearm.dae" />
-            </geometry>
-            <material name="LightGrey">
-                <color rgba="0.7 0.7 0.7 1.0" />
-            </material>
-        </visual>
-        <collision>
-            <origin rpy="1.5707963267948966 0 -1.5707963267948966" xyz="0 0 0.0165" />
-            <geometry>
-                <mesh filename="package://ur5_description/collision/forearm.stl" />
-            </geometry>
-        </collision>
-        <inertial>
-            <mass value="2.275" />
-            <origin rpy="0 1.5707963267948966 0" xyz="-0.196125 0.0 0.0165" />
-            <inertia ixx="0.03121679102890359" ixy="0.0" ixz="0.0" iyy="0.03121679102890359" iyz="0.0" izz="0.004095" />
-        </inertial>
-    </link>
-    <link name="wrist_1_link">
-        <visual>
-            <origin rpy="1.5707963267948966 0 0" xyz="0 0 -0.093" />
-            <geometry>
-                <mesh filename="package://ur5_description/visual/wrist1.dae" />
-            </geometry>
-            <material name="LightGrey">
-                <color rgba="0.7 0.7 0.7 1.0" />
-            </material>
-        </visual>
-        <collision>
-            <origin rpy="1.5707963267948966 0 0" xyz="0 0 -0.093" />
-            <geometry>
-                <mesh filename="package://ur5_description/collision/wrist1.stl" />
-            </geometry>
-        </collision>
-        <inertial>
-            <mass value="1.219" />
-            <origin rpy="0 0 0" xyz="0 0 0" />
-            <inertia ixx="0.0020138887777775" ixy="0.0" ixz="0.0" iyy="0.0020138887777775" iyz="0.0" izz="0.0021942" />
-        </inertial>
-    </link>
-    <link name="wrist_2_link">
-        <visual>
-            <origin rpy="0 0 0" xyz="0 0 -0.095" />
-            <geometry>
-                <mesh filename="package://ur5_description/visual/wrist2.dae" />
-            </geometry>
-            <material name="LightGrey">
-                <color rgba="0.7 0.7 0.7 1.0" />
-            </material>
-        </visual>
-        <collision>
-            <origin rpy="0 0 0" xyz="0 0 -0.095" />
-            <geometry>
-                <mesh filename="package://ur5_description/collision/wrist2.stl" />
-            </geometry>
-        </collision>
-        <inertial>
-            <mass value="1.219" />
-            <origin rpy="0 0 0" xyz="0 0 0" />
-            <inertia ixx="0.0018310388509175" ixy="0.0" ixz="0.0" iyy="0.0018310388509175" iyz="0.0" izz="0.0021942" />
-        </inertial>
-    </link>
-    <link name="wrist_3_link">
-        <visual>
-            <origin rpy="1.5707963267948966 0 0" xyz="0 0 -0.0818" />
-            <geometry>
-                <mesh filename="package://ur5_description/visual/wrist3.dae" />
-            </geometry>
-            <material name="LightGrey">
-                <color rgba="0.7 0.7 0.7 1.0" />
-            </material>
-        </visual>
-        <collision>
-            <origin rpy="1.5707963267948966 0 0" xyz="0 0 -0.0818" />
-            <geometry>
-                <mesh filename="package://ur5_description/collision/wrist3.stl" />
-            </geometry>
-        </collision>
-        <inertial>
-            <mass value="0.1879" />
-            <origin rpy="0 0 0" xyz="0.0 0.0 -0.01525" />
-            <inertia ixx="8.062472608343e-05" ixy="0.0" ixz="0.0" iyy="8.062472608343e-05" iyz="0.0" izz="0.0001321171875" />
-        </inertial>
-    </link>
-    <joint name="base_link-base_link_inertia" type="fixed">
-        <parent link="base_link" />
-        <child link="base_link_inertia" />
-        <origin rpy="0 0 3.141592653589793" xyz="0 0 0" />
-    </joint>
-    <joint name="shoulder_pan_joint" type="revolute">
-        <parent link="base_link_inertia" />
-        <child link="shoulder_link" />
-        <origin rpy="0 0 0" xyz="0 0 0.089159" />
-        <axis xyz="0 0 1" />
-        <limit effort="150.0" lower="-6.283185307179586" upper="6.283185307179586" velocity="3.141592653589793" />
-        <dynamics damping="0" friction="0" />
-    </joint>
-    <joint name="shoulder_lift_joint" type="revolute">
-        <parent link="shoulder_link" />
-        <child link="upper_arm_link" />
-        <origin rpy="1.570796327 0 0" xyz="0 0 0" />
-        <axis xyz="0 0 1" />
-        <limit effort="150.0" lower="-6.283185307179586" upper="6.283185307179586" velocity="3.141592653589793" />
-        <dynamics damping="0" friction="0" />
-    </joint>
-    <joint name="elbow_joint" type="revolute">
-        <parent link="upper_arm_link" />
-        <child link="forearm_link" />
-        <origin rpy="0 0 0" xyz="-0.425 0 0" />
-        <axis xyz="0 0 1" />
-        <limit effort="150.0" lower="-3.141592653589793" upper="3.141592653589793" velocity="3.141592653589793" />
-        <dynamics damping="0" friction="0" />
-    </joint>
-    <joint name="wrist_1_joint" type="revolute">
-        <parent link="forearm_link" />
-        <child link="wrist_1_link" />
-        <origin rpy="0 0 0" xyz="-0.39225 0 0.10915" />
-        <axis xyz="0 0 1" />
-        <limit effort="28.0" lower="-6.283185307179586" upper="6.283185307179586" velocity="3.141592653589793" />
-        <dynamics damping="0" friction="0" />
-    </joint>
-    <joint name="wrist_2_joint" type="revolute">
-        <parent link="wrist_1_link" />
-        <child link="wrist_2_link" />
-        <origin rpy="1.570796327 0 0" xyz="0 -0.09465 -1.941303950897609e-11" />
-        <axis xyz="0 0 1" />
-        <limit effort="28.0" lower="-6.283185307179586" upper="6.283185307179586" velocity="3.141592653589793" />
-        <dynamics damping="0" friction="0" />
-    </joint>
-    <joint name="wrist_3_joint" type="revolute">
-        <parent link="wrist_2_link" />
-        <child link="wrist_3_link" />
-        <origin rpy="1.570796326589793 3.141592653589793 3.141592653589793" xyz="0 0.0823 -1.688001216681175e-11" />
-        <axis xyz="0 0 1" />
-        <limit effort="28.0" lower="-6.283185307179586" upper="6.283185307179586" velocity="3.141592653589793" />
-        <dynamics damping="0" friction="0" />
-    </joint>
-    <link name="base" />
-    <joint name="base_link-base_fixed_joint" type="fixed">
-        <origin rpy="0 0 3.141592653589793" xyz="0 0 0" />
-        <parent link="base_link" />
-        <child link="base" />
-    </joint>
-    <link name="flange" />
-    <joint name="wrist_3-flange" type="fixed">
-        <parent link="wrist_3_link" />
-        <child link="flange" />
-        <origin rpy="0 -1.5707963267948966 -1.5707963267948966" xyz="0 0 0" />
-    </joint>
-    <link name="tool0" />
-    <joint name="flange-tool0" type="fixed">
-        <origin rpy="1.5707963267948966 0 1.5707963267948966" xyz="0 0 0" />
-        <parent link="flange" />
-        <child link="tool0" />
-    </joint>
-    <link name="gripper_link">
-        <inertial>
-          <origin xyz="0 0 0" rpy="0 0 0"/>
-          <mass value="1"/>
-          <inertia ixx="0.0" ixy="0" ixz="0" iyy="0.0" iyz="0" izz="0.0"/>
-        </inertial>
-        <visual>
-          <origin xyz="0 0 0" rpy="0 0 0"/>
-          <geometry>
-            <cylinder radius="0.0425" length="0.26"/>
-          </geometry>
-          <material name="grey">
-            <color rgba="0.5 0.5 0.5 1"/>
-          </material>
-        </visual>
-        <collision>
-          <origin xyz="0 0 0" rpy="0 0 0"/>
-          <geometry>
-            <cylinder radius="0.0525" length="0.27"/>
-          </geometry>
-        </collision>
-    </link>
-    <joint name="joint_tool0_gripper" type="fixed">
-        <parent link="tool0"/>
-        <child link="gripper_link"/>
-        <origin xyz="0.0 0.0 0.13" rpy="0.0 0.0 0.0"/>
-    </joint>
-    <link name="gripper">
-    </link>
-    <joint name="joint_gripper_link_to_gripper" type="fixed">
-        <parent link="gripper_link"/>
-        <child link="gripper"/>
-        <origin xyz="0.0 0.0 0.13" rpy="0.0 0.0 0.0"/>
-    </joint>
-    <link name="world"/>
-    <joint name="joint_fixed" type="fixed">
-        <parent link="world"/>
-        <child link="base_link"/>
-        <origin xyz="0.0 0.0 0.0" rpy="0.0 0.0 0.0"/>
-    </joint>
+    <xacro:include filename="ur5_core.xacro" />
 </robot>
